Commit message: Add hokuyo lidar

File: urdf/mira.urdf (robot description, URDF)
Before this commit: robot mira, 18 links, 17 joints
Links:
- removed link mobile_base_2d_lidar_frame
- removed link mobile_base_lidar_frame
- added link base_laser_front_link, mass 0.16; collision mesh filename=package://sps/meshes/sensors/hokuyo_convex.dae; visual mesh filename=package://sps/meshes/sensors/hokuyo.dae
Joints:
- removed joint mobile_base_2d_lidar_joint
- removed joint mobile_base_lidar_joint
- added joint base_laser_front_hokuyo_urg04_laser_joint: type fixed, parent base_link, child base_laser_front_link, origin xyz=0.2 0 0.21 rpy=0 0 0, axis 0 1 0

File: urdf/mobile_base.xacro (robot description, xacro)
@@ -61,4 +61,5 @@
 		<material>Gazebo/Orange</material>
 	</gazebo>
+	<!--
 	<joint name="${prefix}_lidar_joint" type="fixed">
 	  <origin xyz = "0.285 0 0.12" rpy = "${PI/2} 0 ${PI/2}"/>
@@ -105,4 +106,10 @@
 		<material>Gazebo/Orange</material>
 	</gazebo>
+	-->
 	<xacro:include filename="$(find sps)/urdf/mobile_base_plugin.xacro" />
+    <xacro:include filename="$(find sps)/urdf/sensors/hokuyo_urg04_laser.urdf.xacro"/>
+  <!-- base laser front -->
+  <xacro:hokuyo_urg04_laser name="base_laser_front" parent="base" ros_topic="scan_front" update_rate="10" min_angle="-1.57" max_angle="1.57">
+    <origin xyz="0.2 0 0.21" rpy="0 0 0"/>
+  </xacro:hokuyo_urg04_laser>
 </robot>
